File: Electronics/Conducting-filament/555-test/555-test.sch (KiCad schematic (older format))
At the start: 7 parts, among them J1 Conn_01x02_Male, J2 Conn_01x01_Male, U1 LM555

Commit message: Further work on test circuit.
Parts:
- removed J2: Conn_01x01_Male, Connector_PinHeader_2.54mm:PinHeader_1x01_P2.54mm_Vertical, symbol Connector:Conn_01x01_Male
- added D1: LED, LED_THT:LED_D3.0mm, symbol Device:LED
- added R3: 220R, Resistor_THT:R_Axial_DIN0207_L6.3mm_D2.5mm_P7.62mm_Horizontal, symbol Device:R
Connections:
- net +5V: now also D1.2 (A)
- net at U1.3 (Q): now also R3.2
- new net: D1.1 (K), R3.1
Changed lines of the file:
@@
 	3425 3325 3125 3325
-$Comp
-L Connector:Conn_01x01_Male J2
-U 1 1 62D23357
-P 4525 2325
-F 0 "J2" H 4497 2257 50  0000 R CNN
-F 1 "Conn_01x01_Male" H 4497 2348 50  0000 R CNN
-F 2 "Connector_PinHeader_2.54mm:PinHeader_1x01_P2.54mm_Vertical" H 4525 2325 50  0001 C CNN
-F 3 "~" H 4525 2325 50  0001 C CNN
-	1    4525 2325
-	-1   0    0    1
-$EndComp
 $Comp
 L Device:CP C2
@@
 	1    0    0    -1
 $EndComp
+$Comp
+L Device:R R3
+U 1 1 62DEB696
+P 4325 2175
+F 0 "R3" H 4395 2221 50  0000 L CNN
+F 1 "220R" H 4395 2130 50  0000 L CNN
+F 2 "Resistor_THT:R_Axial_DIN0207_L6.3mm_D2.5mm_P7.62mm_Horizontal" V 4255 2175 50  0001 C CNN
+F 3 "~" H 4325 2175 50  0001 C CNN
+	1    4325 2175
+	1    0    0    -1
+$EndComp
+$Comp
+L Device:LED D1
+U 1 1 62DEBC8B
+P 4325 1875
+F 0 "D1" V 4364 1758 50  0000 R CNN
+F 1 "LED" V 4273 1758 50  0000 R CNN
+F 2 "LED_THT:LED_D3.0mm" H 4325 1875 50  0001 C CNN
+F 3 "~" H 4325 1875 50  0001 C CNN
+	1    4325 1875
+	0    -1   -1   0
+$EndComp
+$Comp
+L power:+5V #PWR0105
+U 1 1 62DEC38D
+P 4325 1725
+F 0 "#PWR0105" H 4325 1575 50  0001 C CNN
+F 1 "+5V" H 4340 1898 50  0000 C CNN
+F 2 "" H 4325 1725 50  0001 C CNN
+F 3 "" H 4325 1725 50  0001 C CNN
+	1    4325 1725
+	1    0    0    -1
+$EndComp
